File: oshpark REV1/penghis_cahn.brd (EAGLE design)
At the start: 99.4 x 99.6 mm, 67 parts, among them IC1 PCF8574T, P0 TPB1,27, P1 TPB1,27, T1 BC847, T2 BC847, U1 MCP73831

Commit message: even more labels
Parts:
- added R19, R20: 300R, rcl:R0603
- moved LED3 8.10 mm to (20.3, 8.13), turned to 180 degrees
- moved R11 0.51 mm to (22.9, 8.13)
Connections:
- new net N$17: R20.1, SAO2.1
- new net N$9: R19.1, SAO1.1
- net NEO_OUT: now also R19.2, R20.2
Routing:
- net NEO_OUT: track 19.5 -> 144.5 mm, vias 0 -> 6
- net N$9: track 0.00 -> 10.1 mm
- net VIN: track 161.8 -> 166.3 mm
- net N$17: track 0.00 -> 3.31 mm
- net N$15: track 5.93 -> 2.64 mm
- net CC1101_CSN_GPIO2: track 34.9 -> 36.5 mm
Other:
- board text added: "AP2112K 3V3 REGULATOR"
- board text added: "CH340C USB SERIAL CONVERTER"
- board text added: "MCP73831 LiPo charger"
