File: oshpark REV1/penghis_cahn.sch (EAGLE design)
At the start: 67 parts, among them IC1 PCF8574T, P0 TPB1,27, P1 TPB1,27, T1 BC847, T2 BC847, U1 MCP73831

Commit message: even more labels
Parts:
- added R19, R20: 300R, rcl:R-EU_R0603
Connections:
- new net N$17: R20.1, SAO2.GPIO1
- new net N$9: R19.1, SAO1.GPIO1
- net NEO_OUT: now also R19.2, R20.2
Changed lines of the file:
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@@
 <part name="SAO1" library="SparkFun-Connectors" deviceset="SAO-SHITTY-ADDON" device="MASTER"/>
 <part name="SAO2" library="SparkFun-Connectors" deviceset="SAO-SHITTY-ADDON" device="MASTER"/>
+<part name="R19" library="rcl" deviceset="R-EU_" device="R0603" value="300R"/>
+<part name="R20" library="rcl" deviceset="R-EU_" device="R0603" value="300R"/>
 </parts>
 <sheets>
@@
 <instance part="SAO1" gate="G$1" x="-5.08" y="134.62"/>
 <instance part="SAO2" gate="G$1" x="30.48" y="134.62"/>
+<instance part="R19" gate="G$1" x="12.7" y="147.32" rot="R90"/>
+<instance part="R20" gate="G$1" x="48.26" y="147.32" rot="R90"/>
 </instances>
 <busses>
@@
 <label x="-7.62" y="40.64" size="1.016" layer="95" xref="yes"/>
 </segment>
+<segment>
+<pinref part="R19" gate="G$1" pin="2"/>
+<wire x1="12.7" y1="152.4" x2="12.7" y2="154.94" width="0.1524" layer="91"/>
+<label x="12.7" y="154.94" size="1.016" layer="95" xref="yes"/>
+</segment>
+<segment>
+<pinref part="R20" gate="G$1" pin="2"/>
+<wire x1="48.26" y1="154.94" x2="48.26" y2="152.4" width="0.1524" layer="91"/>
+<label x="48.26" y="154.94" size="1.016" layer="95" xref="yes"/>
+</segment>
 </net>
 <net name="NEO_IN" class="0">
@@
 </segment>
 </net>
+<net name="N$9" class="0">
+<segment>
+<pinref part="SAO1" gate="G$1" pin="GPIO1"/>
+<pinref part="R19" gate="G$1" pin="1"/>
+<wire x1="2.54" y1="139.7" x2="12.7" y2="139.7" width="0.1524" layer="91"/>
+<wire x1="12.7" y1="139.7" x2="12.7" y2="142.24" width="0.1524" layer="91"/>
+</segment>
+</net>
+<net name="N$17" class="0">
+<segment>
+<pinref part="SAO2" gate="G$1" pin="GPIO1"/>
+<pinref part="R20" gate="G$1" pin="1"/>
+<wire x1="38.1" y1="139.7" x2="48.26" y2="139.7" width="0.1524" layer="91"/>
+<wire x1="48.26" y1="139.7" x2="48.26" y2="142.24" width="0.1524" layer="91"/>
+</segment>
+</net>
